Commit message: feat(add resize palet)

File: sema_ws/src/sema_models/urdf/sema_pallet.urdf (robot description, URDF)
Before this commit: robot sema_pallet, 1 links, 0 joints
Links:
- link sema_pallet_link: geometry collision box size=0.8 1.2 0.144; visual mesh filename=package://sema_models/model/sema_pallet/mesh/sema_pallet.dae scale=1.0 1.0 1.0
