Commit message: feat(cam files ready)

File: sema_ws/src/sema_description/urdf/depthai_camera.xacro (robot description, xacro)
@@ -2,5 +2,5 @@
 <robot xmlns:xacro="http://wiki.ros.org/xacro" name="oak_d">
   <xacro:arg name="camera_name"   default="oak_d_lite"  />
-  <xacro:arg name="camera_model"  default="OAK-D-PRO"  />
+  <xacro:arg name="camera_model"  default="OAK-D-LITE"  />
   <xacro:arg name="base_frame"    default="oak-d_frame" />
   <xacro:arg name="parent_frame"  default="base_link"   />

File: sema_ws/src/sema_description/urdf/macro/depthai_camera_macro.xacro (robot description, xacro)
@@ -1,35 +1,59 @@
 <?xml version="1.0"?>
 <robot xmlns:xacro="http://ros.org/wiki/xacro">
-  <xacro:macro name="depthai_camera" params="camera_name parent base_frame prefix
-                                             camera_model:=OAK-D-LITE
+  <xacro:macro name="depthai_camera" params="camera_name parent prefix
+                                             base_frame:=oak-d_frame camera_model:=OAK-D-POE
                                              x:=0 y:=0 z:=0 R:=0 P:=0 Y:=0
                                              r:=0.8 g:=0.8 b:=0.8 a:=0.8">
-      <!-- https://docs.luxonis.com/projects/hardware/en/latest/ -->
+      <!-- OAK-D cameras info: https://docs.luxonis.com/projects/hardware/en/latest/ -->
+      <xacro:if value="${camera_model=='OAK-D-POE'}">
+        <!-- physical parameters -->
+        <xacro:property name="cam_mass"        value="0.361"  />  <!-- kg -->
+        <xacro:property name="cam_size_x"      value="0.131"  />  <!-- m -->
+        <xacro:property name="cam_size_y"      value="0.031"  />  <!-- m -->
+        <xacro:property name="cam_size_z"      value="0.101"  />  <!-- m -->
+        <xacro:property name="cam_x_col"       value="-0.014" />  <!-- m -->
+        <xacro:property name="cam_y_col"       value="0.0"    />  <!-- m -->
+        <xacro:property name="cam_z_col"       value="-0.018" />  <!-- m -->
+        <!-- vision parameters -->
+        <xacro:property name="base_line"       value="0.075"/> <!-- m -->
+        <xacro:property name="h_fov"           value="1.25664"/> <!-- 72 deg -->
+        <xacro:property name="width"           value="1280"/> <!-- pix -->
+        <xacro:property name="height"          value="800"/> <!-- pix -->
+        <xacro:property name="min_depth_range" value="0.7"/> <!-- m -->
+        <xacro:property name="max_depth_range" value="15"/>  <!-- m -->
+      </xacro:if>
       <xacro:if value="${camera_model=='OAK-D-LITE'}">
-        <xacro:property name="mass"        value="0.061"  />
-        <xacro:property name="size_x"      value="0.091"  />
-        <xacro:property name="size_y"      value="0.0175" />
-        <xacro:property name="size_z"      value="0.028"  />
-        <xacro:property name="delta_x_col" value="-0.006" />
-        <xacro:property name="delta_y_col" value="0.0"    />
-        <xacro:property name="delta_z_col" value="-0.0055"/>
-      </xacro:if>
-      <xacro:if value="${camera_model=='OAK-D-POE'}">
-        <xacro:property name="mass"        value="0.361" />
-        <xacro:property name="size_x"      value="0.131" />
-        <xacro:property name="size_y"      value="0.031" />
-        <xacro:property name="size_z"      value="0.101" />
-        <xacro:property name="delta_x_col" value="-0.014"  />
-        <xacro:property name="delta_y_col" value="0.0"  />
-        <xacro:property name="delta_z_col" value="-0.018"  />
+        <!-- physical parameters -->
+        <xacro:property name="cam_mass"        value="0.061"  />
+        <xacro:property name="cam_size_x"      value="0.091"  />
+        <xacro:property name="cam_size_y"      value="0.0175" />
+        <xacro:property name="cam_size_z"      value="0.028"  />
+        <xacro:property name="cam_x_col"       value="-0.006" />
+        <xacro:property name="cam_y_col"       value="0.0"    />
+        <xacro:property name="cam_z_col"       value="-0.005"/>
+        <!-- vision parameters  -->
+        <xacro:property name="base_line"       value="0.075"/>
+        <xacro:property name="h_fov"           value="1.27409"/> <!-- 73° -->
+        <xacro:property name="width"           value="640"/>
+        <xacro:property name="height"          value="480"/>
+        <xacro:property name="min_depth_range" value="0.35"/>
+        <xacro:property name="max_depth_range" value="10"/>
       </xacro:if>
       <xacro:if value="${camera_model=='OAK-D-PRO'}">
-        <xacro:property name="mass"        value="0.091" />
-        <xacro:property name="size_x"      value="0.097" />
-        <xacro:property name="size_y"      value="0.0235" />
-        <xacro:property name="size_z"      value="0.0295" />
-        <xacro:property name="delta_x_col" value="-0.01"  />
-        <xacro:property name="delta_y_col" value="0.0"  />
-        <xacro:property name="delta_z_col" value="-0.0055"  />
+        <!-- physical parameters -->
+        <xacro:property name="cam_mass"        value="0.091"  />
+        <xacro:property name="cam_size_x"      value="0.097"  />
+        <xacro:property name="cam_size_y"      value="0.0235" />
+        <xacro:property name="cam_size_z"      value="0.0295" />
+        <xacro:property name="cam_x_col"       value="-0.01"  />
+        <xacro:property name="cam_y_col"       value="0.0"    />
+        <xacro:property name="cam_z_col"       value="-0.005"/>
+        <!-- vision parameters -->
+        <xacro:property name="base_line"       value="0.075"/>
+        <xacro:property name="h_fov"           value="1.2566"/> <!-- 72° -->
+        <xacro:property name="width"           value="1280"/>
+        <xacro:property name="height"          value="800"/>
+        <xacro:property name="min_depth_range" value="0.7"/>
+        <xacro:property name="max_depth_range" value="15"/>
       </xacro:if>
       <!-- base_link of the sensor -->
@@ -45,15 +69,15 @@
           </visual>
           <collision name="${camera_name}_collision">
-              <origin xyz="${delta_x_col} ${delta_y_col} ${delta_z_col}" rpy="0.0 0.0 ${pi/2}"/>
+              <origin xyz="${cam_x_col} ${cam_y_col} ${cam_z_col}" rpy="0.0 0.0 ${pi/2}"/>
               <geometry>
-                  <box size="${size_x} ${size_y} ${size_z}"/>
+                  <box size="${cam_size_x} ${cam_size_y} ${cam_size_z}"/>
               </geometry>
           </collision>
           <inertial>
-            <mass value="${mass}"/>
+            <mass value="${cam_mass}"/>
             <inertia
-              ixx="${mass*(size_y*size_y+size_z*size_z)/12}"
-              iyy="${mass*(size_x*size_x+size_z*size_z)/12}"
-              izz="${mass*(size_x*size_x+size_y*size_y)/12}"
+              ixx="${cam_mass*(cam_size_y*cam_size_y+cam_size_z*cam_size_z)/12}"
+              iyy="${cam_mass*(cam_size_x*cam_size_x+cam_size_z*cam_size_z)/12}"
+              izz="${cam_mass*(cam_size_x*cam_size_x+cam_size_y*cam_size_y)/12}"
               ixy="0"
               ixz="0"
@@ -73,13 +97,13 @@
           <child link="${prefix}${camera_name}_rgb_camera_optical_frame"/>
       </joint>
-      <!-- Gazebo camera setup -->
-      <gazebo reference="${prefix}${base_frame}">
+    <!-- Gazebo camera setup -->
+    <gazebo reference="${prefix}${base_frame}">
       <sensor type="depth" name="${prefix}${camera_name}_sensor">
         <update_rate>18.0</update_rate>
         <camera name="${prefix}${camera_name}_camera">
-          <horizontal_fov>1.20427718388</horizontal_fov>
+          <horizontal_fov>${h_fov}</horizontal_fov>
           <image>
-            <width>640</width>
-            <height>480</height>
+            <width>${5*width/8}</width>
+            <height>${5*height/8}</height>
             <format>R8G8B8</format>
           </image>
@@ -98,9 +122,8 @@
         </camera>
         <plugin name="depth_camera_plugin_${camera_name}" filename="libgazebo_ros_openni_kinect.so">
-          <!-- Oak D LITE camera data: https://docs.luxonis.com/projects/hardware/en/latest/pages/DM9095.html -->
           <!-- plugin config data: https://classic.gazebosim.org/tutorials?tut=ros_depth_camera&cat=connect_ros -->
-          <baseline>0.075</baseline>
-          <pointCloudCutoff>0.35</pointCloudCutoff>
-          <pointCloudCutoffMax>10.0</pointCloudCutoffMax>
+          <baseline>${base_line}</baseline>
+          <pointCloudCutoff>${min_depth_range}</pointCloudCutoff>
+          <pointCloudCutoffMax>${max_depth_range}</pointCloudCutoffMax>
           <alwaysOn>true</alwaysOn>
           <updateRate>0.0</updateRate>
@@ -113,13 +136,8 @@
           <frameName>${prefix}${camera_name}_rgb_camera_optical_frame</frameName>
           <distortionK1>0.00000001</distortionK1>
-	  <distortionK2>0.00000001</distortionK2>
-	  <distortionK3>0.00000001</distortionK3>
-	  <distortionT1>0.00000001</distortionT1>
-	  <distortionT2>0.00000001</distortionT2>
-	  <CxPrime>0</CxPrime>
-	  <Cx>0</Cx>
-	  <Cy>0</Cy>
-	  <focalLength>0</focalLength>
-	  <hackBaseline>0</hackBaseline>
+          <distortionK2>0.00000001</distortionK2>
+          <distortionK3>0.00000001</distortionK3>
+          <distortionT1>0.00000001</distortionT1>
+          <distortionT2>0.00000001</distortionT2>
         </plugin>
       </sensor>

File: sema_ws/src/sema_description/urdf/sema.xacro (robot description, xacro)
@@ -107,25 +107,14 @@
   <!-- add Depth camera model and plugin  -->
   <xacro:if value="$(arg oak_d_enabled)">
-    <!--
-    <xacro:include filename="$(find sema_description)/urdf/macro/oak_d_macro.xacro"/>
-    <xacro:oak_d name="$(arg dc_name)" prefix="$(arg prefix)"/>
-    <joint name="$(arg prefix)$(arg dc_name)ee_joint" type="fixed">
-      <origin xyz="0.12 0 0" rpy="-${pi} -${pi/2} 0"/>
-      <parent link="$(arg prefix)wrist_3_link"/>
-      <child link="$(arg prefix)$(arg dc_name)base_link"/>
-    </joint>
-    -->
     <xacro:arg name="camera_name"   default="oak" />
     <xacro:arg name="camera_model"  default="OAK-D-LITE" />
-    <xacro:arg name="base_frame"    default="oak-d_frame" />
     <xacro:arg name="parent_frame"  default="$(arg prefix)wrist_3_link" />
-    <xacro:arg name="cam_pos_x"     default="0.12" />
-    <xacro:arg name="cam_pos_y"     default="0.0" />
-    <xacro:arg name="cam_pos_z"     default="0.0" />
+    <xacro:arg name="cam_pos_x"     default="0.08" />
     <xacro:arg name="cam_roll"      default="-${pi}" />
     <xacro:arg name="cam_pitch"     default="-${pi/2}" />
-    <xacro:arg name="cam_yaw"       default="0.0" />
     <xacro:include filename="$(find sema_description)/urdf/macro/depthai_camera_macro.xacro"/>
-    <xacro:depthai_camera camera_name = "$(arg camera_name)" parent = "$(arg parent_frame)" camera_model = "$(arg camera_model)" base_frame = "$(arg base_frame)" cam_pos_x = "$(arg cam_pos_x)" cam_pos_y = "$(arg cam_pos_y)" cam_pos_z = "$(arg cam_pos_z)" cam_roll = "$(arg cam_roll)" cam_pitch = "$(arg cam_pitch)" cam_yaw = "$(arg cam_yaw)"/>
+    <xacro:depthai_camera camera_name = "$(arg camera_name)" parent = "$(arg parent_frame)"
+                          camera_model = "$(arg camera_model)" prefix = "$(arg prefix)"
+                          x = "$(arg cam_pos_x)" R = "$(arg cam_roll)" P = "$(arg cam_pitch)"/>
   </xacro:if>
 </robot>
