Commit message: feat(add depens)

File: sema_ws/src/sema_description/urdf/macro/depthai_camera_macro.xacro (robot description, xacro)
@@ -5,8 +5,4 @@
                                            cam_roll cam_pitch cam_yaw
                                            r:=0.8 g:=0.8 b:=0.8 a:=0.8">
-    <xacro:property name="M_PI"     value="3.1415926535897931" />
-    <xacro:property name="model"    value="${camera_model}" />
-    <!-- <xacro:if value="${model == 'BW1098OAK'}">
-    </xacro:if> -->
     <xacro:property name="baseline" value="0.075" />
     <!-- base_link of the sensor -->
@@ -22,5 +18,5 @@
             <origin xyz="0 0 0" rpy="0 0 0"/>
             <geometry>
-                <mesh filename="package://depthai_bridge/urdf/models/${model}.stl" />
+                <mesh filename="package://depthai_bridge/urdf/models/${camera_model}.stl" />
             </geometry>
             <material name="mat">
@@ -34,4 +30,14 @@
             </geometry>
         </collision>
+        <inertial>
+          <mass value="0.4"/>
+          <inertia
+            ixx="0.0002046"
+            iyy="0.000095"
+            izz="0.0002046"
+            ixy="0"
+            ixz="0"
+            iyz="0"/>
+        </inertial>
     </link>
     <joint name="${camera_name}_model_origin_joint" type="fixed">
@@ -49,9 +55,9 @@
     <link name="${camera_name}_rgb_camera_optical_frame"/>
     <joint name="${camera_name}_rgb_camera_optical_joint" type="fixed">
-        <origin xyz="0 0 0" rpy="-${M_PI/2} 0.0 -${M_PI/2}"/>
+        <origin xyz="0 0 0" rpy="-${pi/2} 0.0 -${pi/2}"/>
         <parent link="${camera_name}_rgb_camera_frame"/>
         <child link="${camera_name}_rgb_camera_optical_frame"/>
     </joint>
-    <!-- Gazebo camera setup
+    <!-- Gazebo camera setup -->
     <gazebo reference="${camera_name}_rgb_camera_frame">
       <sensor type="depth" name="${camera_name}_sensor">
@@ -70,7 +76,9 @@
           <noise>
             <type>gaussian</type>
+             <!--
              Noise is sampled independently per pixel on each frame.
              That pixel's noise value is added to each of its color
               channels, which at that point lie in the range [0,1].
+              -->
             <mean>0.0</mean>
             <stddev>0.007</stddev>
@@ -78,6 +86,8 @@
         </camera>
         <plugin name="depth_camera_plugin_${camera_name}" filename="libgazebo_ros_openni_kinect.so">
+           <!--
            Oak D LITE camera data: https://docs.luxonis.com/projects/hardware/en/latest/pages/DM9095.html
            plugin config data: https://classic.gazebosim.org/tutorials?tut=ros_depth_camera&cat=connect_ros
+           -->
           <baseline>0.075</baseline>
           <alwaysOn>true</alwaysOn>
@@ -100,5 +110,4 @@
       </sensor>
     </gazebo>
-    -->
 </xacro:macro>
 </robot>

Commit message: update

File: sema_ws/src/sema_description/urdf/macro/depthai_camera_macro.xacro (robot description, xacro)
@@ -75,4 +75,5 @@
           </collision>
           <inertial>
+            <origin xyz="${cam_x_col} ${cam_y_col} ${cam_z_col}" rpy="0.0 0.0 ${pi/2}"/>
             <mass value="${cam_mass}"/>
             <inertia
